File: SEM15.kicad_sch (KiCad schematic)
At the start: 60 parts, among them J1 Conn_01x04, J2 Conn_01x01_Male, J3 Conn_01x01_Male, J4 Conn_01x01_Male, J5 Conn_01x01_Male, J6 Conn_01x01_Male, J7 Conn_01x01_Male, Q1 AO3401A, Q2 AO3401A, Q3 AO3401A, Q4 AO3401A, SW1 SW_DPST_x2, T1 Tab, U1 STC8G1K08-SOP16

Commit message: fix
Parts:
- D11, D13, D14, D15, D17, D18, D19, D20, D22, D23, D24: value LED -> LED_G
- SW1: footprint sajat:magasgomb -> sajat:SW_Push_TS-1187A
Changed lines of the file:
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@@
       (effects (font (size 1.27 1.27)))
     )
-    (property "Value" "LED" (at 180.34 38.1 90)
+    (property "Value" "LED_G" (at 180.34 38.1 90)
       (effects (font (size 1.27 1.27)))
     )
@@
       (effects (font (size 1.27 1.27)))
     )
-    (property "Value" "LED" (at 142.24 37.592 90)
+    (property "Value" "LED_G" (at 142.24 37.592 90)
       (effects (font (size 1.27 1.27)))
     )
@@
       (effects (font (size 1.27 1.27)))
     )
-    (property "Value" "LED" (at 145.542 38.862 90)
+    (property "Value" "LED_G" (at 145.542 38.862 90)
       (effects (font (size 1.27 1.27)))
     )
@@
       (effects (font (size 1.27 1.27)))
     )
-    (property "Value" "LED" (at 215.9 38.1 90)
+    (property "Value" "LED_G" (at 215.9 38.1 90)
       (effects (font (size 1.27 1.27)))
     )
@@
       (effects (font (size 1.27 1.27)))
     )
-    (property "Value" "LED" (at 189.23 38.1 90)
+    (property "Value" "LED_G" (at 189.23 38.1 90)
       (effects (font (size 1.27 1.27)))
     )
@@
       (effects (font (size 1.27 1.27)))
     )
-    (property "Value" "LED" (at 198.12 38.1 90)
+    (property "Value" "LED_G" (at 198.12 38.1 90)
       (effects (font (size 1.27 1.27)))
     )
@@
       (effects (font (size 1.27 1.27)))
     )
-    (property "Footprint" "sajat:magasgomb" (at 167.894 167.386 0)
+    (property "Footprint" "sajat:SW_Push_TS-1187A" (at 167.894 167.386 0)
       (effects (font (size 1.27 1.27)) hide)
     )
@@
       (effects (font (size 1.27 1.27)))
     )
-    (property "Value" "LED" (at 160.274 39.878 90)
+    (property "Value" "LED_G" (at 160.274 39.878 90)
       (effects (font (size 1.27 1.27)))
     )
@@
       (effects (font (size 1.27 1.27)))
     )
-    (property "Value" "LED" (at 171.958 38.608 90)
+    (property "Value" "LED_G" (at 171.958 38.608 90)
       (effects (font (size 1.27 1.27)))
     )
@@
       (effects (font (size 1.27 1.27)))
     )
-    (property "Value" "LED" (at 154.686 35.56 90)
+    (property "Value" "LED_G" (at 154.686 35.56 90)
       (effects (font (size 1.27 1.27)))
     )
@@
       (effects (font (size 1.27 1.27)))
     )
-    (property "Value" "LED" (at 128.778 37.084 90)
+    (property "Value" "LED_G" (at 128.778 37.084 90)
       (effects (font (size 1.27 1.27)))
     )
@@
       (effects (font (size 1.27 1.27)))
     )
-    (property "Value" "LED" (at 207.01 38.1 90)
-      (effects (font (size 1.27 1.27)))
-    )
+    (property "Value" "LED_G" (at 207.01 38.1 90)
+      (effects (font (size 1.27 1.27)))
+    )
