File: SEM15.kicad_pcb (KiCad board)
At the start: 2 copper layers, 213.5 x 50.2 mm, 53 parts, among them J1 Conn_01x04, Q1 AO3401A, Q2 AO3401A, Q3 AO3401A, Q4 AO3401A, SW1 SW_DPST_x2, U1 STC8G1K08-SOP16

Commit message: rogzitok
Parts:
- added J2: Conn_01x01_Male, Connector_PinHeader_2.54mm:PinHeader_1x01_P2.54mm_Vertical, F.Cu at (150.0, 71.5)
- added J3: Conn_01x01_Male, Connector_PinHeader_2.54mm:PinHeader_1x01_P2.54mm_Vertical, F.Cu at (36.6, 28.5)
- added J4: Conn_01x01_Male, Connector_PinHeader_2.54mm:PinHeader_1x01_P2.54mm_Vertical, F.Cu at (105.5, 71.5)
- added J5: Conn_01x01_Male, Connector_PinHeader_2.54mm:PinHeader_1x01_P2.54mm_Vertical, F.Cu at (219.0, 71.5)
- added J6: Conn_01x01_Male, Connector_PinHeader_2.54mm:PinHeader_1x01_P2.54mm_Vertical, F.Cu at (105.5, 28.5)
- added J7: Conn_01x01_Male, Connector_PinHeader_2.54mm:PinHeader_1x01_P2.54mm_Vertical, F.Cu at (219.0, 28.5)
- added J8: Conn_01x01_Male, Connector_PinHeader_2.54mm:PinHeader_1x01_P2.54mm_Vertical, F.Cu at (36.5, 71.5)
- added J9: Conn_01x01_Male, Connector_PinHeader_2.54mm:PinHeader_1x01_P2.54mm_Vertical, F.Cu at (150.0, 28.5)
- moved SW1 0.29 mm to (30.9, 62.0)
Other:
- outline, holes or cut-outs redrawn

Commit message: Panelizalas, BOM elkezdve.
Parts:
- removed J2, J5, J7, J9: Conn_01x01_Male, Connector_PinHeader_2.54mm:PinHeader_1x01_P2.54mm_Vertical
- moved D12 51.0 mm to (130.1, 78.4)
- moved D15 51.0 mm to (130.1, 58.1)
- moved D18 51.0 mm to (144.1, 68.5)
- moved D21 51.0 mm to (130.1, 68.8)
- moved R9 51.0 mm to (155.6, 91.5)
- moved C3 51.0 mm to (80.3, 73.5)
- moved L4 51.0 mm to (93.5, 89.6)
- moved R11 51.0 mm to (100.5, 89.4)
- moved BT1 51.0 mm to (77.0, 72.6)
- moved D1 51.0 mm to (87.0, 61.0)
- moved D10 51.0 mm to (108.0, 79.0)
- moved D11 51.0 mm to (86.0, 84.0)
- moved D13 51.0 mm to (104.0, 84.0)
- moved D14 51.0 mm to (122.0, 84.0)
- moved D17 51.0 mm to (141.3, 84.0)
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Routing:
- net GND: vias 1 -> 0
Other:
- board size 213.5 x 50.2 mm -> 98 x 50 mm
- board text removed: "Teteje"

Commit message: uj gomb, kivagas
Parts:
- added J2: Conn_01x01_Male, Connector_PinHeader_2.54mm:PinHeader_1x01_P2.54mm_Vertical, F.Cu at (100.0, 52.0)
- added J5: Conn_01x01_Male, Connector_PinHeader_2.54mm:PinHeader_1x01_P2.54mm_Vertical, F.Cu at (130.0, 52.0)
- C3: value C -> 100n
- C4: value C -> 10u
- R12, R7: value R -> 510
- R5, R8: value R -> 1k
- SW1: footprint sajat:SW_Push_K2-1102SP -> sajat:magasgomb
- moved J3 0.50 mm to (82.6, 51.0)
- moved J4 0.50 mm to (151.5, 93.0)
- moved J6 0.50 mm to (151.5, 51.0)
- moved J8 0.50 mm to (82.5, 93.0)
- turned SW1 to 180 degrees
Routing:
- net /SW_IN: track 71.6 -> 66.7 mm
- net /LED_EN_E: track 19.8 -> 22.4 mm, vias 0 -> 2
- net /LED_EN_M7: track 49.8 -> 50.7 mm
- net /P3.1: track 18.4 -> 17.7 mm, vias 2 -> 1
- added copper zone on B.Cu, net GND
Other:
- board size 98 x 50 mm -> 96.5 x 46 mm

Commit message: gerberek, bom
Parts:
- added T1: Tab, kikit:Tab, F.Cu at (166.3, 59.2)
- added T1: Tab, kikit:Tab, F.Cu at (166.3, 84.0)
- added T1: Tab, kikit:Tab, F.Cu at (82.6, 95.3)
- added T1: Tab, kikit:Tab, F.Cu at (151.6, 95.3)
- added T1: Tab, kikit:Tab, F.Cu at (69.2, 59.6)
- added T1: Tab, kikit:Tab, F.Cu at (82.6, 48.6)
- added T1: Tab, kikit:Tab, F.Cu at (151.6, 48.6)
- added T1: Tab, kikit:Tab, F.Cu at (69.0, 84.0)
Other:
- board text added: "Készült a SEM 15. születésnapja alkalmából 2008-2023"
- board text added: "M32 By: Dávid P., Kristóf H., Regi R."

Commit message: fix
Parts:
- D11, D13, D14, D15, D17, D18, D19, D20, D22, D23, D24: value LED -> LED_G
- SW1: footprint sajat:magasgomb -> sajat:SW_Push_TS-1187A
Changed lines of the file:
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@@
         (effects (font (size 1 1) (thickness 0.15)))
     )
-    (fp_text value "LED" (at 0 1.65) (layer "F.Fab")
+    (fp_text value "LED_G" (at 0 1.65) (layer "F.Fab")
         (effects (font (size 1 1) (thickness 0.15)))
     )
@@
         (effects (font (size 1 1) (thickness 0.15)))
     )
-    (fp_text value "LED" (at 0 1.65) (layer "F.Fab")
+    (fp_text value "LED_G" (at 0 1.65) (layer "F.Fab")
         (effects (font (size 1 1) (thickness 0.15)))
     )
@@
         (effects (font (size 1 1) (thickness 0.15)))
     )
-    (fp_text value "LED" (at 0 1.65) (layer "F.Fab")
+    (fp_text value "LED_G" (at 0 1.65) (layer "F.Fab")
         (effects (font (size 1 1) (thickness 0.15)))
     )
@@
         (effects (font (size 1 1) (thickness 0.15)))
     )
-    (fp_text value "LED" (at 0 1.65) (layer "F.Fab")
+    (fp_text value "LED_G" (at 0 1.65) (layer "F.Fab")
         (effects (font (size 1 1) (thickness 0.15)))
     )
@@
         (effects (font (size 1 1) (thickness 0.15)))
     )
-    (fp_text value "LED" (at 0 1.65) (layer "F.Fab")
+    (fp_text value "LED_G" (at 0 1.65) (layer "F.Fab")
         (effects (font (size 1 1) (thickness 0.15)))
     )
@@
     )
   )
-  (footprint "sajat:magasgomb" (layer "F.Cu")
+  (footprint "sajat:SW_Push_TS-1187A" (layer "F.Cu")
     (at 76.95 83.95 180)
     (property "Sheetfile" "SEM15.kicad_sch")
@@
         (effects (font (size 1 1) (thickness 0.15)))
     )
-    (fp_text user "${REFERENCE}" (at -5.95 0.275 90) (layer "F.Fab")
+    (fp_text user "${REFERENCE}" (at -5.95 0.275 270) (layer "F.Fab")
         (effects (font (size 1 1) (thickness 0.15)))
     )
@@
         (effects (font (size 1 1) (thickness 0.15)))
     )
-    (fp_text value "LED" (at 0 1.65 90) (layer "F.Fab")
+    (fp_text value "LED_G" (at 0 1.65 90) (layer "F.Fab")
         (effects (font (size 1 1) (thickness 0.15)))
     )
@@
         (effects (font (size 1 1) (thickness 0.15)))
     )
-    (fp_text value "LED" (at 0 1.65 90) (layer "F.Fab")
+    (fp_text value "LED_G" (at 0 1.65 90) (layer "F.Fab")
         (effects (font (size 1 1) (thickness 0.15)))
     )
@@
         (effects (font (size 1 1) (thickness 0.15)))
     )
-    (fp_text value "LED" (at 0 1.65) (layer "F.Fab")
+    (fp_text value "LED_G" (at 0 1.65) (layer "F.Fab")
         (effects (font (size 1 1) (thickness 0.15)))
     )
@@
         (effects (font (size 1 1) (thickness 0.15)))
     )
-    (fp_text value "LED" (at 0 1.65 90) (layer "F.Fab")
+    (fp_text value "LED_G" (at 0 1.65 90) (layer "F.Fab")
         (effects (font (size 1 1) (thickness 0.15)))
     )
@@
         (effects (font (size 1 1) (thickness 0.15)))
     )
-    (fp_text value "LED" (at 0 1.65 90) (layer "F.Fab")
+    (fp_text value "LED_G" (at 0 1.65 90) (layer "F.Fab")
         (effects (font (size 1 1) (thickness 0.15)))
     )
@@
         (effects (font (size 1 1) (thickness 0.15)))
     )
-    (fp_text value "LED" (at 0 1.65) (layer "F.Fab")
-        (effects (font (size 1 1) (thickness 0.15)))
-    )
+    (fp_text value "LED_G" (at 0 1.65) (layer "F.Fab")
+        (effects (font (size 1 1) (thickness 0.15)))
+    )

Commit message: sent to jlc
Parts:
- added J2: Conn_01x01_Male, Connector_PinHeader_2.54mm:PinHeader_1x01_P2.54mm_Vertical, F.Cu at (80.7, 161.4)
- added J5: Conn_01x01_Male, Connector_PinHeader_2.54mm:PinHeader_1x01_P2.54mm_Vertical, F.Cu at (149.7, 161.4)
- added J7: Conn_01x01_Male, Connector_PinHeader_2.54mm:PinHeader_1x01_P2.54mm_Vertical, F.Cu at (149.7, 119.4)
- added J9: Conn_01x01_Male, Connector_PinHeader_2.54mm:PinHeader_1x01_P2.54mm_Vertical, F.Cu at (80.7, 119.4)
- added T1: Tab, kikit:Tab, F.Cu at (149.8, 163.8)
- added T1: Tab, kikit:Tab, F.Cu at (67.2, 153.4)
- added T1: Tab, kikit:Tab, F.Cu at (67.2, 127.4)
- added T1: Tab, kikit:Tab, F.Cu at (80.8, 163.8)
- added T1: Tab, kikit:Tab, F.Cu at (80.8, 117.0)
- added T1: Tab, kikit:Tab, F.Cu at (149.8, 117.0)
- added T1: Tab, kikit:Tab, F.Cu at (164.6, 127.8)
- added T1: Tab, kikit:Tab, F.Cu at (164.8, 153.4)
Routing:
- net GND: track 0.00 -> 7.19 mm
- net (no net): vias 0 -> 1
Other:
- board size 96.5 x 46 mm -> 98.3 x 114.4 mm
